File: servo-drive-brd.sch (KiCad schematic (older format))
At the start: 9 parts, among them CON1 BARREL_JACK, P1 CONN_01X03, U1 LM555N

Commit message: Final version (hopefully, fingers crossed) with a linear power regulator, and a horizontally mounted pot (facing the right way)
Parts:
- added C3, C4: 10 uF, Capacitors_ThroughHole:C_Radial_D5_L11_P2, symbol CP
- added U2, U3: LM7805CT, TO-220, symbol LM7805CT
- renumbered PTV09A-2~-TOP to PTV09A-2
Connections:
- net +5V: now also P1.2 (P2), C4.1, U3.3 (OUT); no longer CON1.1, P1.1 (P1)
- net GND: now also C3.2, C4.2, U3.2 (GND)
- net at U1.3 (Q): now also P1.1 (P1); no longer P1.2 (P2)
- new net: C3.1, CON1.1, U3.1 (IN)
- no-connect marks 1 -> 0
Changed lines of the file:
@@
 L R R1
 U 1 1 56AAEA01
-P 7350 3200
-F 0 "R1" V 7430 3200 50  0000 C CNN
-F 1 "56K" V 7350 3200 50  0000 C CNN
-F 2 "Resistors_ThroughHole:Resistor_TO-220_Vertical" V 7280 3200 50  0001 C CNN
-F 3 "" H 7350 3200 50  0000 C CNN
-	1    7350 3200
+P 7350 3050
+F 0 "R1" V 7430 3050 50  0000 C CNN
+F 1 "56K" V 7350 3050 50  0000 C CNN
+F 2 "Resistors_ThroughHole:Resistor_TO-220_Vertical" V 7280 3050 50  0001 C CNN
+F 3 "" H 7350 3050 50  0000 C CNN
+	1    7350 3050
 	1    0    0    -1
 $EndComp
@@
 $EndComp
 $Comp
-L POT PTV09A-2~-TOP
+L POT PTV09A-2
 U 1 1 56AAF04E
 P 7350 3750
-F 0 "PTV09A-2 -TOP" H 7350 3650 50  0000 C CNN
+F 0 "PTV09A-2" H 7350 3650 50  0000 C CNN
 F 1 "POT 100K" H 7350 3750 50  0000 C CNN
 F 2 "local_lib:PTV09A-2-TOP" H 7350 3750 50  0001 C CNN
@@
 	1    0    0    -1
 $EndComp
-Wire Wire Line
-	7350 3350 7350 3500
-Wire Wire Line
-	6400 3750 7200 3750
-Connection ~ 7050 3750
-Wire Wire Line
-	6400 4050 7050 4050
-Wire Wire Line
-	6800 4200 7050 4200
-Wire Wire Line
-	5900 4500 8300 4500
-Connection ~ 6750 3750
-Wire Wire Line
-	6400 3950 6400 4200
-Connection ~ 6750 4050
-Wire Wire Line
-	6900 4050 6900 4200
-Connection ~ 6900 4200
-Connection ~ 6900 4050
 $Comp
 L GND #PWR02
@@
 L +5V #PWR03
 U 1 1 56AAFAFA
-P 7350 2950
-F 0 "#PWR03" H 7350 2800 50  0001 C CNN
-F 1 "+5V" H 7350 3090 50  0000 C CNN
-F 2 "" H 7350 2950 50  0000 C CNN
-F 3 "" H 7350 2950 50  0000 C CNN
-	1    7350 2950
-	1    0    0    -1
-$EndComp
-Wire Wire Line
-	7350 2950 7350 3050
-Wire Wire Line
-	5400 3950 5050 3950
-Wire Wire Line
-	5050 3950 5050 3000
-Wire Wire Line
-	5050 3000 8300 3000
-Connection ~ 7350 3000
-Wire Wire Line
-	6900 4500 6900 4600
-Connection ~ 6900 4500
+P 7350 2800
+F 0 "#PWR03" H 7350 2650 50  0001 C CNN
+F 1 "+5V" H 7350 2940 50  0000 C CNN
+F 2 "" H 7350 2800 50  0000 C CNN
+F 3 "" H 7350 2800 50  0000 C CNN
+	1    7350 2800
+	1    0    0    -1
+$EndComp
 $Comp
 L BARREL_JACK CON1
 U 1 1 56AAFB98
-P 8600 3100
-F 0 "CON1" H 8600 3350 50  0000 C CNN
-F 1 "BARREL_JACK" H 8600 2900 50  0000 C CNN
-F 2 "Connect:BARREL_JACK" H 8600 3100 50  0001 C CNN
-F 3 "" H 8600 3100 50  0000 C CNN
-	1    8600 3100
-	-1   0    0    -1
+P 3000 2950
+F 0 "CON1" H 3000 3200 50  0000 C CNN
+F 1 "BARREL_JACK" H 3000 2750 50  0000 C CNN
+F 2 "Connect:BARREL_JACK" H 3000 2950 50  0001 C CNN
+F 3 "" H 3000 2950 50  0000 C CNN
+	1    3000 2950
+	1    0    0    -1
 $EndComp
 $Comp
@@
 $EndComp
 Wire Wire Line
-	7850 3550 7850 4500
+	6400 3750 7200 3750
+Connection ~ 7050 3750
+Wire Wire Line
+	6400 4050 7050 4050
+Wire Wire Line
+	6800 4200 7050 4200
+Wire Wire Line
+	3300 4500 7850 4500
+Connection ~ 6750 3750
+Wire Wire Line
+	6400 3950 6400 4200
+Connection ~ 6750 4050
+Wire Wire Line
+	6900 4050 6900 4200
+Connection ~ 6900 4200
+Connection ~ 6900 4050
+Wire Wire Line
+	7350 2800 7350 2900
+Wire Wire Line
+	5050 3950 5400 3950
+Wire Wire Line
+	5050 2850 5050 3950
+Wire Wire Line
+	4650 2850 7750 2850
+Connection ~ 7350 2850
+Wire Wire Line
+	6900 4500 6900 4600
+Connection ~ 6900 4500
+Wire Wire Line
+	7850 4500 7850 3550
 Connection ~ 7050 4500
-Wire Wire Line
-	8300 4500 8300 3100
 Connection ~ 7850 4500
 Wire Wire Line
-	6400 3450 7850 3450
-Wire Wire Line
-	6400 3450 6400 3550
-NoConn ~ 7350 3450
-Connection ~ 8300 3200
-Wire Wire Line
-	7850 3000 7850 3350
-Connection ~ 7850 3000
+	6400 3350 6400 3550
 Wire Wire Line
 	6400 4200 5300 4200
@@
 Connection ~ 6400 4050
 Wire Wire Line
-	5900 3350 5900 3000
-Connection ~ 5900 3000
-Wire Wire Line
-	5900 4150 5900 4500
+	5900 2850 5900 3350
+Connection ~ 5900 2850
+Wire Wire Line
+	5900 4500 5900 4150
 Connection ~ 6800 4500
+Wire Wire Line
+	7750 3450 7850 3450
+Wire Wire Line
+	7750 2850 7750 3450
+Connection ~ 7750 2850
+Wire Wire Line
+	6400 3350 7850 3350
+Wire Wire Line
+	3300 2850 3850 2850
+Wire Wire Line
+	3300 2950 3300 4500
+Wire Wire Line
+	3300 3150 4700 3150
+Connection ~ 3300 3050
+Connection ~ 5900 4500
+Connection ~ 3300 3150
+Connection ~ 5050 2850
+Wire Wire Line
+	7350 3200 7350 3500
+$Comp
+L LM7805CT U2
+U 1 1 56D7541B
+P -117100 -93900
+F 0 "U2" H -117300 -93700 50  0000 C CNN
+F 1 "LM7805CT" H -117100 -93700 50  0000 L CNN
+F 2 "TO-220" H -117100 -93800 50  0000 C CIN
+F 3 "" H -117100 -93900 50  0000 C CNN
+	1    -117100 -93900
+	1    0    0    -1
+$EndComp
+$Comp
+L LM7805CT U3
+U 1 1 56D75992
+P 4250 2900
+F 0 "U3" H 4050 3100 50  0000 C CNN
+F 1 "LM7805CT" H 4250 3100 50  0000 L CNN
+F 2 "TO-220" H 4250 3000 50  0000 C CIN
+F 3 "" H 4250 2900 50  0000 C CNN
+	1    4250 2900
+	1    0    0    -1
+$EndComp
+$Comp
+L CP C3
+U 1 1 56D75B1F
+P 3650 3000
+F 0 "C3" H 3675 3100 50  0000 L CNN
+F 1 "10 uF" H 3675 2900 50  0000 L CNN
+F 2 "Capacitors_ThroughHole:C_Radial_D5_L11_P2" H 3688 2850 50  0001 C CNN
+F 3 "" H 3650 3000 50  0000 C CNN
+	1    3650 3000
+	1    0    0    -1
+$EndComp
+$Comp
+L CP C4
+U 1 1 56D75B6E
+P 4700 3000
+F 0 "C4" H 4725 3100 50  0000 L CNN
+F 1 "10 uF" H 4725 2900 50  0000 L CNN
+F 2 "Capacitors_ThroughHole:C_Radial_D5_L11_P2" H 4738 2850 50  0001 C CNN
+F 3 "" H 4700 3000 50  0000 C CNN
+	1    4700 3000
+	1    0    0    -1
+$EndComp
+Connection ~ 4250 3150
+Connection ~ 3650 2850
+Connection ~ 4700 2850
+Connection ~ 4700 3150
+Connection ~ 3650 3150
+Connection ~ 3850 2850
+Connection ~ 4650 2850
+Connection ~ 3300 2850
+Connection ~ 3300 2950
 $EndSCHEMATC
